File: W65C51_LudaCris.kicad_sch (KiCad schematic)
At the start: 45 parts, among them J1 USB_RST, J2 USB_C, J3 I2C, J4 RS-232, J5 USB_Status, J6 I2C, J7 I2C, U1 W65C51NxP, U10 74HC191, U11 ATF22V10, U12 ATF22V10, U13 74HC138, U14 74HC283, U17 MCP2221AxP, U18 MAX232, U19 74HC191, U4 74HC191, U5 74HC191, U6 1.8432 MHz, U8 74HC573, U9 74HC191

Commit message: GAL PLD
Parts:
- removed C13, C14, C15, C16, C18, C19, C20, C21, C22: 100nF, symbol Device:C
- removed J1: USB_RST, Connector_PinHeader_2.54mm:PinHeader_1x02_P2.54mm_Horizontal, symbol Connector_Generic:Conn_01x02
- removed J2: USB_C, Connector_USB:USB_C_Plug_JAE_DX07P024AJ1, symbol Connector:USB_B
- removed J3, J6: I2C, Connector_PinHeader_2.54mm:PinHeader_1x04_P2.54mm_Horizontal, symbol Connector_Generic:Conn_01x04
- removed J4: RS-232, symbol Connector:DE9_Receptacle
- removed J5: USB_Status, Connector_PinHeader_2.54mm:PinHeader_1x06_P2.54mm_Horizontal, symbol Connector_Generic:Conn_01x06
- removed J7: I2C, Connector_PinHeader_2.54mm:PinHeader_1x03_P2.54mm_Horizontal, symbol Connector_Generic:Conn_01x03
- removed R2, R3, R4: 3.3K, symbol Device:R
- removed U17: MCP2221AxP, Package_DIP:DIP-14_W7.62mm, symbol W65C51_LudaCris:MCP2221AxP
- removed U18: MAX232, Package_DIP:DIP-16_W7.62mm_Socket, symbol W65C51_LudaCris:MAX232
- removed U6: 1.8432 MHz, Oscillator:Oscillator_DIP-8, symbol Oscillator:KC2520Z
- added BAR1, BAR2, BAR3: LED-Array-8, Package_DIP:DIP-16_W7.62mm, symbol W65C51_LudaCris:LED-Array-8
- added C12: 10uF, Capacitor_THT:CP_Radial_D4.0mm_P1.50mm, symbol Device:C_Polarized
- added C7: 100nF, Capacitor_THT:C_Disc_D3.4mm_W2.1mm_P2.50mm, symbol Device:C
- added H1, H2, H3: MountingHole_Pad, MountingHole:MountingHole_3.2mm_M3_Pad, symbol Mechanical:MountingHole_Pad
- added RN1, RN2, RN3: 220, Resistor_THT:R_Array_SIP9, symbol Device:R_Network08
- added U12: 74AHC240, symbol 74xx:74AHC240
- C1: renamed from C12; footprint (none) -> Capacitor_THT:C_Disc_D3.4mm_W2.1mm_P2.50mm
- C10, C11, C8, C9: footprint (none) -> Capacitor_THT:C_Disc_D3.4mm_W2.1mm_P2.50mm
- C13: renamed from C1; footprint (none) -> Capacitor_THT:C_Disc_D3.4mm_W2.1mm_P2.50mm
- C2: value 470n -> 100nF; footprint (none) -> Capacitor_THT:C_Disc_D3.4mm_W2.1mm_P2.50mm
- C3, C4, C5, C6: value 1uF -> 100nF; footprint (none) -> Capacitor_THT:C_Disc_D3.4mm_W2.1mm_P2.50mm
- R1: footprint (none) -> Resistor_THT:R_Axial_DIN0207_L6.3mm_D2.5mm_P7.62mm_Horizontal
- U4: renamed from U12; footprint Package_DIP:DIP-24_W7.62mm -> Package_DIP:DIP-24_W7.62mm_Socket
- U5: renamed from U11; footprint Package_DIP:DIP-24_W7.62mm -> Package_DIP:DIP-24_W7.62mm_Socket
- renumbered U14 to U10, U4 to U11, U13 to U2, U8 to U3, U19 to U6, U5 to U7, U10 to U8
Connections:
- net CLK: now also U4.1 (CLK/IN)
- net CR0: now also BAR1.1 (A), BAR3.1 (A)
- net CR1: now also BAR1.2 (A), BAR3.2 (A)
- net CR2: now also BAR1.3 (A), BAR3.3 (A)
- net CR3: now also BAR1.4 (A), BAR3.4 (A)
- net CR4: now also BAR1.5 (A), BAR3.5 (A)
- net CR5: now also BAR1.6 (A), BAR3.6 (A)
- net CR6: now also BAR1.7 (A), BAR3.7 (A)
- net CR7: now also BAR1.8 (A), BAR3.8 (A)
- net CTL_REG_WR: now also U12.17 (2A0); no longer U3.11 (Load), U4.17 (I/O), U5.15 (I/O)
- net GND: now also C3.2, C4.2, U4.13 (IN), U5.1 (CLK/IN), U5.6 (IN), U5.7 (IN), C12.2, C7.2, H1.1, H2.1, H3.1, RN1.1 (common), RN2.1 (common), RN3.1 (common), U12.1 (1OE), U12.10 (GND), U12.19 (2OE); no longer U1.16 (~{DCD}), U1.9 (~{CTS}), U4.9 (IN)
- net VCC: now also C2.1, C3.1, C4.1, C5.1, C6.1, U7.16 (VCC), U9.16 (VCC), C12.1, C7.1, U12.20 (VCC); no longer U1.2 (CS1), U2.6 (E2), U4.1 (CLK/IN), U5.1 (CLK/IN)
- net ~{BAUD_CLK}: now also U4.8 (IN), U12.8 (1A3); no longer U4.13 (IN)
- net ~{BAUD_LOAD}: now also U12.13 (2A2)
- net ~{CTEN}: now also U12.15 (2A1); no longer U5.14 (I/O)
- net ~{CTL_REG_WR}: now also U12.2 (1A0)
- net ~{DSR}: now also U12.11 (2A3)
- net ~{TX_COMPLETE}: now also U4.9 (IN), U12.6 (1A2); no longer U4.8 (IN)
- net ~{TX_START}: now also U12.4 (1A1)
- net ~{DTR}: now reaches U1.11 (~{DTR})
- net RxC: now reaches U1.5 (RxC)
- net XTAL2: now reaches U1.7 (XTAL2)
- net ~{RTS}: now reaches U1.8 (~{RTS})
- net A0 renamed RS0
- net A1 renamed RS1
- net ~{IOCS1} renamed ~{CS2}
- net ~{IRQ1} renamed ~{IRQ}
- net ~{WR} renamed R~{W}
- new net: BAR1.9 (K), RN1.2 (R1)
- new net: BAR1.10 (K), RN1.3 (R2)
- new net: BAR1.11 (K), RN1.4 (R3)
- new net: BAR1.12 (K), RN1.5 (R4)
- new net: BAR1.13 (K), RN1.6 (R5)
- new net: BAR1.14 (K), RN1.7 (R6)
- new net: BAR1.15 (K), RN1.8 (R7)
- new net: BAR1.16 (K), RN1.9 (R8)
- new net: BAR2.1 (A), U12.18 (1Y0)
- new net: BAR2.10 (K), RN2.3 (R2)
- new net: BAR2.11 (K), RN2.4 (R3)
- new net: BAR2.12 (K), RN2.5 (R4)
- new net: BAR2.13 (K), RN2.6 (R5)
- new net: BAR2.14 (K), RN2.7 (R6)
- new net: BAR2.15 (K), RN2.8 (R7)
- new net: BAR2.16 (K), RN2.9 (R8)
- new net: BAR2.2 (A), U12.16 (1Y1)
- new net: BAR2.3 (A), U12.14 (1Y2)
- new net: BAR2.4 (A), U12.12 (1Y3)
- new net: BAR2.5 (A), U12.3 (2Y0)
- new net: BAR2.6 (A), U12.5 (2Y1)
- new net: BAR2.7 (A), U12.7 (2Y2)
- new net: BAR2.8 (A), U12.9 (2Y3)
- new net: BAR2.9 (K), RN2.2 (R1)
- new net: BAR3.10 (K), RN3.3 (R2)
- new net: BAR3.11 (K), RN3.4 (R3)
- new net: BAR3.12 (K), RN3.5 (R4)
- new net: BAR3.13 (K), RN3.6 (R5)
- new net: BAR3.14 (K), RN3.7 (R6)
- new net: BAR3.15 (K), RN3.8 (R7)
- new net: BAR3.16 (K), RN3.9 (R8)
- new net: BAR3.9 (K), RN3.2 (R1)
- new net CS1: U1.2 (CS1), U2.6 (E2)
- new net CTL_REG_LOAD: U3.11 (Load), U4.17 (I/O)
- new net ~{CTS}: U1.9 (~{CTS})
- new net ~{DCD}: U1.16 (~{DCD})
- no-connect marks 50 -> 37
Other:
- note added: "~{BAUD_LOAD} = ~{BAUD_CLK} AND ~{TX_START}"
- note added: "~{CTEN} = ! ~{DSR}"
- note added: "~{DSR} Set Hi by ~{TX_START} Falling Edge Set Lo (Active) by ~{TX_COMPLETE} Falling Edge"
- note removed: "W65C51 Ctrl Reg"
- note removed: "~{BAUD_LOAD} = ~{BAUD_CLOCK} AND ~{TX_START}"
- note removed: "~{DSR} Set Hi by ~{TX_START} Falling Edge Set Lo by ~{TX_COMPLETE} Falling Edge"

Commit message: PCB 2.54mm centres
Parts:
- removed BAR2, BAR3: LED-Array-8, Package_DIP:DIP-16_W7.62mm, symbol W65C51_LudaCris:LED-Array-8
- removed RN2, RN3: 220, Resistor_THT:R_Array_SIP9, symbol Device:R_Network08
- removed U12: 74AHC240, symbol 74xx:74AHC240
- added H4: MountingHole_Pad, MountingHole:MountingHole_3.2mm_M3_Pad, symbol Mechanical:MountingHole_Pad
- BAR1: footprint Package_DIP:DIP-16_W7.62mm -> Package_DIP:DIP-16_W7.62mm_Socket
Connections:
- net CR0: now also BAR1.8 (A), U3.12 (Q7); no longer BAR1.1 (A), U3.19 (Q0)
- net CR1: now also BAR1.7 (A), U3.13 (Q6); no longer BAR1.2 (A), U3.18 (Q1)
- net CR2: now also BAR1.6 (A), U3.14 (Q5); no longer BAR1.3 (A), U3.17 (Q2)
- net CR3: now also BAR1.5 (A), U3.15 (Q4); no longer BAR1.4 (A), U3.16 (Q3)
- net CR4: now also U3.16 (Q3); no longer BAR1.5 (A), U3.15 (Q4)
- net CR5: now also BAR1.4 (A), U3.17 (Q2); no longer BAR1.6 (A), U3.14 (Q5)
- net CR6: now also BAR1.3 (A), U3.18 (Q1); no longer BAR1.7 (A), U3.13 (Q6)
- net CR7: now also BAR1.2 (A), U3.19 (Q0); no longer BAR1.8 (A), U3.12 (Q7)
- net CTL_REG_WR: now also BAR1.1 (A)
- net D0: now also U3.9 (D7); no longer U3.2 (D0)
- net D1: now also U3.8 (D6); no longer U3.3 (D1)
- net D2: now also U3.7 (D5); no longer U3.4 (D2)
- net D3: now also U3.6 (D4); no longer U3.5 (D3)
- net D4: now also U3.5 (D3); no longer U3.6 (D4)
- net D5: now also U3.4 (D2); no longer U3.7 (D5)
- net D6: now also U3.3 (D1); no longer U3.8 (D6)
- net D7: now also U3.2 (D0); no longer U3.9 (D7)
- net GND: now also H4.1
Other:
- moved on the sheet: BAR1, H1, H2, H3, RN1

Commit message: pcb
Parts:
- added J1, J2: Conn_01x14, Connector_PinHeader_2.54mm:PinHeader_1x14_P2.54mm_Vertical, symbol W65C51_LudaCris:Conn_01x14_2.54mm
Connections:
- net CLK: now also J2.2 (Pin_2)
- net CS1: now also J1.2 (Pin_2)
- net D0: now also J2.11 (Pin_11)
- net D1: now also J2.10 (Pin_10)
- net D2: now also J2.9 (Pin_9)
- net D3: now also J2.8 (Pin_8)
- net D4: now also J2.7 (Pin_7)
- net D5: now also J2.6 (Pin_6)
- net D6: now also J2.5 (Pin_5)
- net D7: now also J2.4 (Pin_4)
- net GND: now also J1.1 (Pin_1)
- net RS0: now also J1.13 (Pin_13)
- net RS1: now also J1.14 (Pin_14)
- net RxC: now also J1.5 (Pin_5)
- net RxD: now also J1.12 (Pin_12)
- net R~{W}: now also J2.1 (Pin_1)
- net TxD: now also J1.10 (Pin_10)
- net VCC: now also J2.14 (Pin_14)
- net XTAL1: now also J1.6 (Pin_6)
- net XTAL2: now also J1.7 (Pin_7)
- net ~{CS2}: now also J1.3 (Pin_3)
- net ~{CTS}: now also J1.9 (Pin_9)
- net ~{DCD}: now also J2.13 (Pin_13)
- net ~{DSR}: now also J2.12 (Pin_12)
- net ~{DTR}: now also J1.11 (Pin_11)
- net ~{IRQ}: now also J2.3 (Pin_3)
- net ~{RES}: now also J1.4 (Pin_4)
- net ~{RTS}: now also J1.8 (Pin_8)
